Commit message: Decrese size of imu module and add body_length to change from squre to rectangle.

File: quadruped/urdf/quadruped_model.xacro (robot description, xacro)
@@ -9,8 +9,10 @@
   <xacro:property name="scaling_factor" value="2.2" />
   <!--height:z width:y width:x -->
+  <xacro:property name="body_length" value="${scaling_factor*0.208}" />
   <xacro:property name="body_width" value="${scaling_factor*0.108}" />
   <xacro:property name="body_height" value="${scaling_factor*0.055}" />
   <xacro:property name="body_mass" value="${(scaling_factor**3)*0.4}" />
-  <xacro:property name="imu_size" value="${scaling_factor*0.02}" />
+  <!-- we donot want a small object upon the robot body -->
+  <xacro:property name="imu_size" value="0.00001" />
   <xacro:property name="imu_mass" value="${(scaling_factor**3)*0.05}" />
   <!--height:z width:y depth:x -->
@@ -70,5 +72,5 @@
     <visual>
       <geometry>
-        <box size="${body_width} ${body_width} ${body_height}"/>
+        <box size="${body_length} ${body_width} ${body_height}"/>
       </geometry>
       <material name="black"/>
@@ -76,8 +78,8 @@
     <collision>
       <geometry>
-        <box size="${body_width} ${body_width} ${body_height}"/>
+        <box size="${body_length} ${body_width} ${body_height}"/>
       </geometry>
     </collision>
-    <xacro:box_inertial mass="${body_mass}" width="${body_width}" depth="${body_width}"/>
+    <xacro:box_inertial mass="${body_mass}" width="${body_length}" depth="${body_width}"/>
   </link>
   <joint name="dummy_base_joint" type="fixed">
@@ -274,5 +276,5 @@
       <parent link="base_link"/>
       <child link="${prefix}_${suffix}_leg3"/>
-      <origin xyz="${reflect_right*body_width/2.0} ${reflect_front*body_width/2.0} 0" rpy="0 0 ${reflect_front*pi/2.0 - reflect_front*reflect_right*pi/4.0}"/>
+      <origin xyz="${reflect_right*body_length/2.0} ${reflect_front*body_width/2.0} 0" rpy="0 0 ${reflect_front*pi/2.0 - reflect_front*reflect_right*pi/4.0}"/>
       <limit lower="${leg3_joint_low}" upper="${leg3_joint_high}" effort="${servo_effort_limit}" velocity="${servo_vel}"/>
       <dynamics friction="0.0" />

Commit message: Change robot color and configuration and add joint controller publisher.

File: quadruped/urdf/quadruped_model.xacro (robot description, xacro)
@@ -11,5 +11,5 @@
   <xacro:property name="body_length" value="${scaling_factor*0.208}" />
   <xacro:property name="body_width" value="${scaling_factor*0.108}" />
-  <xacro:property name="body_height" value="${scaling_factor*0.055}" />
+  <xacro:property name="body_height" value="${scaling_factor*0.1}" />
   <xacro:property name="body_mass" value="${(scaling_factor**3)*0.4}" />
   <!-- we donot want a small object upon the robot body -->
@@ -21,12 +21,12 @@
   <xacro:property name="leg1_depth" value="${scaling_factor*0.015}" />
   <xacro:property name="leg1_mass" value="${(scaling_factor**3)*0.8}" />
-  <xacro:property name="leg1_joint_low" value="${-pi*2.0/18.0}" />
-  <xacro:property name="leg1_joint_high" value="${pi*2.0/18.0}" />
+  <xacro:property name="leg1_joint_low" value="${-pi*2.0}" />
+  <xacro:property name="leg1_joint_high" value="${pi*2.0}" />
   <xacro:property name="leg2_height" value="${scaling_factor*0.025}" />
   <xacro:property name="leg2_width" value="${scaling_factor*0.01}" />
   <xacro:property name="leg2_depth" value="${scaling_factor*0.1}" />
   <xacro:property name="leg2_mass" value="${(scaling_factor**3)*0.05}" />
-  <xacro:property name="leg2_joint_low" value="${-pi*2.0/18.0}" />
-  <xacro:property name="leg2_joint_high" value="${pi*2.0/18.0}" />
+  <xacro:property name="leg2_joint_low" value="${-pi*2.0}" />
+  <xacro:property name="leg2_joint_high" value="${pi*2.0}" />
   <xacro:property name="leg2_init_pitch" value="${pi*16.0/18.0}" />
   <xacro:property name="leg3_height" value="${scaling_factor*0.052}" />
@@ -34,6 +34,6 @@
   <xacro:property name="leg3_depth" value="${scaling_factor*0.015}" />
   <xacro:property name="leg3_mass" value="${(scaling_factor**3)*0.1}" />
-  <xacro:property name="leg3_joint_low" value="${-pi*2.0/18.0}" />
-  <xacro:property name="leg3_joint_high" value="${pi*2.0/18.0}" />
+  <xacro:property name="leg3_joint_low" value="${-pi*2.0}" />
+  <xacro:property name="leg3_joint_high" value="${pi*2.0}" />
   <xacro:property name="leg_tip_mass" value="${(scaling_factor**3)*0.02}" />
   <xacro:property name="servo_vel" value="4.0" />
@@ -91,5 +91,5 @@
     <mu1>100000.0</mu1>
     <mu2>100000.0</mu2>
-    <material>Gazebo/Black</material>
+    <material>Gazebo/White</material>
   </gazebo>
   <gazebo reference="dummy_base_joint">
@@ -200,5 +200,5 @@
           <box size="${leg1_depth} ${leg1_width} ${leg1_height}"/>
         </geometry>
-        <material name="black"/>
+        <material name="white"/>
       </visual>
       <collision>
@@ -252,5 +252,5 @@
       <mu1>100000.0</mu1>
       <mu2>100000.0</mu2>
-      <material>Gazebo/Black</material>
+      <material>Gazebo/White</material>
     </gazebo>
   </xacro:macro>
@@ -276,5 +276,5 @@
       <parent link="base_link"/>
       <child link="${prefix}_${suffix}_leg3"/>
-      <origin xyz="${reflect_right*body_length/2.0} ${reflect_front*body_width/2.0} 0" rpy="0 0 ${reflect_front*pi/2.0 - reflect_front*reflect_right*pi/4.0}"/>
+      <origin xyz="${reflect_right*body_length/2.0} ${reflect_front*body_width/2.0} ${-(body_height/2.0)}" rpy="0 0 ${reflect_front*pi/2.0 - reflect_front*reflect_right*pi/4.0}"/>
       <limit lower="${leg3_joint_low}" upper="${leg3_joint_high}" effort="${servo_effort_limit}" velocity="${servo_vel}"/>
       <dynamics friction="0.0" />
@@ -283,5 +283,5 @@
       <mu1>100000.0</mu1>
       <mu2>100000.0</mu2>
-      <material>Gazebo/White</material>
+      <material>Gazebo/Black</material>
     </gazebo>
   </xacro:macro>
